File: Hardware/Jig/Qwiic_Spectral_Sensor-AS7265x-BottomJig.sch (EAGLE design)
At the start: 51 parts, among them J2 Serial Interface, J5 Flash Programming, J8 PTH, U1 AS72651, U3 4MB Flash, U5 AS72653, U6 AS72652

Commit message: Silk changes before panelization
Parts:
- removed C1: 1.0uF, SparkFun-Capacitors:1.0UF-0603-16V-10%
- removed C2, C4, C6: 0.1uF, SparkFun-Capacitors:0.1UF-0603-25V-(+80/-20%)
- removed C3, C5, C7: 10uF, SparkFun-Capacitors:10UF-0603-6.3V-20%
- removed D1: BLUE, SparkFun-LED:LED-BLUE0603
- removed D2: 5700k, SparkFun-LED:LED-WHITE3014
- removed D3: IR, SparkFun-LED:LED-IR0603
- removed D4: RED, SparkFun-LED:LED-RED0603
- removed D5: UV, SparkFun-LED:LED-UVPLCC
- removed FD1, FD2, FD3, FD4: FIDUCIAL1X2, SparkFun-Aesthetics:FIDUCIAL1X2
- removed J1, J4: (no value), SparkFun-Connectors:QWIIC_CONNECTORJS-1MM
- removed JP1: JUMPER-SMT_3_2-NC_TRACE_SILK, SparkFun-Jumpers:JUMPER-SMT_3_2-NC_TRACE_SILK
- removed JP2: JUMPER-SMT_2_NO_SILK, SparkFun-Jumpers:JUMPER-SMT_2_NO_SILK
- removed JP3, JP4, JP5: JUMPER-SMT_2_NC_TRACE_NO-SILK, SparkFun-Jumpers:JUMPER-SMT_2_NC_TRACE_NO-SILK
- removed R10, R11, R12, R9: 2.2k, SparkFun-Resistors:2.2KOHM-0603-1/10W-1%
- removed R7, R8: 10k, SparkFun-Resistors:10KOHM-0603-1/10W-1%
- removed TP1: TEST-POINT3, SparkFun-Connectors:TEST-POINT3
- removed U5: AS72653, Qwiic_Spectral_Sensor-AS7265x:AS72653
- removed U6: AS72652, Qwiic_Spectral_Sensor-AS7265x:AS72652
- added BUTTON1, BUTTON2: CAPSENSE_BUTTON_PAD_ONLY, Testing:CAPSENSE_BUTTON_PAD_ONLY
- added FRAME2: FRAME-LEDGER, SparkFun-Aesthetics:FRAME-LEDGER
- added H5, H6: STAND-OFF, SparkFun-Hardware:STAND-OFF
- added J_SCL, J_SCL1, J_SCL2, J_SCL3, J_SCL4, J_SCL5, J_SDA, J_SDA1: JUMPER-SMT_2_NO_NO-SILK, SparkFun-Jumpers:JUMPER-SMT_2_NO_NO-SILK
- added MT_FAIL, MT_PASS, PROGRAM, PT_FAIL, PT_PASS, S0, S1, S2, S3, S4: (no value), Testing:LED1206
- added R6: 330, SparkFun-Resistors:330OHM-0603-1/10W-1%
- added U2: 74LVC4066, Testing:74LVC4066_MUX_1:1_X4
- R1, R3, R4, R5: value 10k -> 330; device SparkFun-Resistors:10KOHM-0603-1/10W-1% -> SparkFun-Resistors:330OHM-0603-1/10W-1%
- R2: value 1k -> 330; device SparkFun-Resistors:1KOHM-0603-1/10W-1% -> SparkFun-Resistors:330OHM-0603-1/10W-1%
- U1: value AS72651 -> FLYING_JALAPENO; device Qwiic_Spectral_Sensor-AS7265x:AS72651 -> Testing:FLYING_JALAPENO_V3MALE
- U3: value 4MB Flash -> 74LVC4066; device SparkFun-IC-Memory:AT25SF041 -> Testing:74LVC4066_MUX_1:1_X4
Connections:
- removed net !RST-ADDR: U1.ADDR, U6.!RST
- removed net I2C_ENB: JP2.2, R3.1, TP1.1, U1.I2C_ENB
- removed net N$1: D4.C, R2.2
- removed net N$11: D5.A, JP3.1
- removed net N$12: R8.2, U5.!CS_SD
- removed net N$13: R7.2, U5.MISO
- removed net N$2: D1.C, U1.LED_IND
- removed net N$3: R5.2, U6.!CS_SD
- removed net N$4: JP1.3, R12.2
- removed net N$5: JP1.1, R11.2
- removed net N$6: D2.A, JP4.1
- removed net N$8: D3.A, JP5.1
- removed net N$9: R1.2, U6.MISO
- removed net SCL_S: R9.1, U1.SCL_M, U5.SCL_S, U6.SCL_S
- removed net SDA_S: R10.1, U1.SDA_M, U5.SDA_S, U6.SDA_S
- new net 3.3V_POWER: U1.V1, U2.VCC, U3.VCC
- new net 5V_POWER: U1.V2
- new net JALAPENO_CS: J_SDA1.1, U1.53(SS), U3.4Y
- new net JALAPENO_I2C_EN: U1.22, U2.1E, U2.2E
- new net JALAPENO_MISO: J_SCL5.1, U1.50(MISO), U3.1Y
- new net JALAPENO_MOSI: J_SCL3.1, U1.51(MOSI), U3.2Y
- new net JALAPENO_RX1-I: J_SDA.1, U1.19(RX1/INT4), U2.4Y
- new net JALAPENO_SCK: J_SCL4.1, U1.52(SCK), U3.3Y
- new net JALAPENO_SCL: J_SCL.1, U1.21(SCL/INT2), U2.2Y
- new net JALAPENO_SDA: J_SCL2.1, U1.20(SDA/INT3), U2.1Y
- new net JALAPENO_SERIAL_EN: U1.23, U2.3E, U2.4E
- new net JALAPENO_SPI_EN: U3.1E, U3.2E, U3.3E, U3.4E
- new net JALAPENO_TX1-O: J_SCL1.1, U1.18(TX1/INT5), U2.3Y
- new net J_24: U1.24
- new net J_25: U1.25
- new net J_26: U1.26
- new net J_27: U1.27
- new net J_28: U1.28
- new net J_29: U1.29
- new net J_30: U1.30
- new net J_A0: U1.A0
- new net J_A1: U1.A1
- new net J_A2: U1.A2
- new net J_A3: U1.A3
- new net J_A4: U1.A4
- new net J_PWM2: U1.2(INT0)
- new net J_PWM3: U1.3(INT1)
- new net J_PWM4: U1.4
- new net J_PWM5: U1.5
- new net N$10: PT_FAIL.A, U1.42/PT_FAIL
- new net N$14: MT_PASS.A, U1.41/PASS
- new net N$15: MT_FAIL.A, U1.40/FAIL
- new net N$16: BUTTON2.CAPSENSE, U1.CAP_PAD2
- new net N$17: BUTTON1.CAPSENSE, U1.CAP_PAD1
- new net N$18: R1.2, U1.12
- new net N$19: PROGRAM.A, R1.1
- new net N$20: R6.2, U1.7
- new net N$21: R5.2, U1.8
- new net N$22: R4.2, U1.9
- new net N$23: R3.2, U1.10
- new net N$24: R2.2, U1.11
- new net N$25: R6.1, S4.A
- new net N$26: R5.1, S3.A
- new net N$27: R4.1, S2.A
- new net N$28: R3.1, S1.A
- new net N$29: R2.1, S0.A
- new net N$7: PT_PASS.A, U1.43/PT_PASS
- new net TARGET_CS: J_SDA1.2, U3.4Z
- new net TARGET_MISO: J_SCL5.2, U3.1Z
- new net TARGET_MOSI: J_SCL3.2, U3.2Z
- new net TARGET_RX: J_SCL1.2, U2.3Z
- new net TARGET_SCK: J_SCL4.2, U3.3Z
- new net TARGET_SCL: J_SCL.2, U2.2Z
- new net TARGET_SDA: J_SCL2.2, U2.1Z
- new net TARGET_TX: J_SDA.2, U2.4Z
- net !CS_EE: no longer U1.!CS_EE, U3.!CS
- net !INT: no longer U1.!INT
- net !RST: no longer R4.1, U1.!RST, U5.!RST
- net 3.3V: no longer C1.1, C2.1, C3.1, C4.1, C5.1, C6.1, C7.1, D1.A, D4.A, J1.2, J4.2, JP1.2, JP3.2, JP4.2, JP5.2, R10.2, R3.2, R4.2, R9.2, U1.VDD, U3.!HOLD(D3), U3.!WP(D2), U3.VCC, U5.VDD, U6.VDD
- net GND: now also MT_FAIL.C, MT_PASS.C, PROGRAM.C, PT_FAIL.C, PT_PASS.C, S0.C, S1.C, S2.C, S3.C, S4.C, U2.GND; no longer C1.2, C2.2, C3.2, C4.2, C5.2, C6.2, C7.2, J1.1, J4.1, JP2.1, R1.1, R2.1, R5.1, R7.1, R8.1, U5.GND, U6.GND
- net LED_DRV: no longer D2.C, U1.LED_DRV
- net LED_DRV1: no longer D3.C, U6.LED_DRV
- net LED_DRV2: no longer D5.C, U5.LED_DRV
- net MISO: no longer U1.MISO, U3.SO(D1)
- net MOSI: no longer U1.MOSI, U3.SI(D0)
- net RX/SCL: no longer J1.4, J4.4, R11.1, U1.RX/SCL
- net SCK: no longer U1.SCK, U3.SCK
- net TX/SDA: no longer J1.3, J4.3, R12.1, U1.TX/SDA
Other:
- note added: "-->"
- note added: "Flying Jalapeno"
- moved on the sheet: BULB1, BULB2, BULB3, J2, J3, J5, J8, R1, R2, R3, R4, R5

Commit message: Intermediate committ. Probably ignore the jig files.
Parts:
- removed BUTTON1: CAPSENSE_BUTTON_PAD_ONLY, Testing:CAPSENSE_BUTTON_PAD_ONLY
- removed PROGRAM, S0, S1, S2, S3, S4: (no value), Testing:LED1206
- removed R1, R2, R3, R4, R5, R6: 330, SparkFun-Resistors:330OHM-0603-1/10W-1%
- added H1, H3, H7: STAND-OFF, SparkFun-Hardware:STAND-OFF
- added TP1: TEST-POINTPOGO_PTH, SparkFun-Connectors:TEST-POINTPOGO_PTH
- J5: device SparkFun-Connectors:AVR_SPI_PROG_3X2TESTPOINTS -> SparkFun-Connectors:AVR_SPI_PROG_3X2NS
Connections:
- net N$16 renamed BUTTON2
- removed net N$17: BUTTON1.CAPSENSE, U1.CAP_PAD1
- removed net N$18: R1.2, U1.12
- removed net N$19: PROGRAM.A, R1.1
- removed net N$20: R6.2, U1.7
- removed net N$21: R5.2, U1.8
- removed net N$22: R4.2, U1.9
- removed net N$23: R3.2, U1.10
- removed net N$24: R2.2, U1.11
- removed net N$25: R6.1, S4.A
- removed net N$26: R5.1, S3.A
- removed net N$27: R4.1, S2.A
- removed net N$28: R3.1, S1.A
- removed net N$29: R2.1, S0.A
- new net I2C_ENB: TP1.1
- net GND: no longer PROGRAM.C, S0.C, S1.C, S2.C, S3.C, S4.C
Other:
- note removed: "-->"
- moved on the sheet: BULB1, BULB2, BULB3
