File: Hardware/Qwiic_Spectral_Sensor-AS7265x.brd (EAGLE design)
At the start: 35.6 x 40.6 mm, 94 parts, among them J2 Serial Interface, J5 Flash Programming, J8 PTH, U1 AS72651, U2 4MB Flash, U3 AS72652, U4 AS72653

Commit message: Remvoing gerbers. Removing jig files. Rename datasheet. Clean up repo before post.
Parts:
- added FRAME3: FRAME-LETTER, SparkFun-Retired:CREATIVE_COMMONS
Changed lines of the file:
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@@
 <attribute name="VALUE" x="5.08" y="26.797" size="0.6096" layer="27" font="vector" ratio="20" align="top-center"/>
 </element>
+<element name="FRAME3" library="SparkFun-Retired" package="CREATIVE_COMMONS" value="FRAME-LETTER" x="-11.43" y="-40.64" smashed="yes"/>
 </elements>
 <signals>
